Commit message: add robot urdf

File: urdf/urdf_test.urdf (robot description, URDF)
Before this commit: robot test_robot, 2 links, 1 joints
Links:
- added link back_ball_link; visual sphere radius=0.05
- added link left_wheel_link; visual cylinder length=0.04 radius=0.072
- added link right_wheel_link; visual cylinder length=0.04 radius=0.072
- link body_link: geometry visual box size=0.4 0.3 0.1
Joints:
- added joint back_ball_joint: type fixed, parent body_link, child back_ball_link, origin xyz=-0.23 0 -0.05 rpy=0 0 0
- added joint left_wheel_joint: type fixed, parent body_link, child left_wheel_link, origin xyz=0 0.18 0 rpy=-1.5707 0 0
- added joint right_wheel_joint: type fixed, parent body_link, child right_wheel_link, origin xyz=0 -0.18 0 rpy=-1.5707 0 0
- joint body_joint: origin (none) -> xyz=0 0 0.1 rpy=0 0 0
