Commit message: robotに色を付けた

File: xacro/diff_drive_robot.urdf.xacro (robot description, xacro)
@@ -1,66 +1,13 @@
 <?xml version="1.0"?>
 <robot name="diff_drive" xmlns:xacro="http://www.ros.org/wiki/xacro">
-    <!-- Base Link -->
-    <link name="base_link">
-        <collision>
-            <origin xyz="-0.151427 -0 0.5" rpy="0 0 0" />
-            <geometry>
-                <box size="2.01142 1 0.568726" />
-            </geometry>
-        </collision>
-        <visual>
-            <origin xyz="-0.151427 -0 0.5" rpy="0 0 0" />
-            <geometry>
-                <box size="2.01142 1 0.568726" />
-            </geometry>
-            <material name="orange" />
-        </visual>
-        <inertial>
-            <origin xyz="-0.151427 -0 0.5" rpy="0 0 0" />
-            <mass value="1.14395" />
-            <inertia
-                ixx="0.126164"
-                ixy="0.0"
-                ixz="0.0"
-                iyy="0.416519"
-                iyz="0.0"
-                izz="0.481014" />
-        </inertial>
-    </link>
     <xacro:include filename="$(find ouagv_robot_description)/xacro/wheel.urdf.xacro" />
     <xacro:include filename="$(find ouagv_robot_description)/xacro/ros2_control.xacro" />
+    <xacro:include filename="$(find ouagv_robot_description)/xacro/body.urdf.xacro" />
+    <xacro:include filename="$(find ouagv_robot_description)/xacro/caster.urdf.xacro" />
+    <xacro:body />
     <xacro:wheel prefix="left" parent="base_link" xyz="0.554283 0.625029 0.3" rpy="-1.5707 0 0" />
     <xacro:wheel prefix="right" parent="base_link" xyz="0.554283 -0.625029 0.3" rpy="-1.5707 0 0" />
+    <xacro:caster parent="base_link" />
     <xacro:diff_drive_control left_joint="left_wheel_joint" right_joint="right_wheel_joint" />
-    <joint name="caster_joint" type="fixed">
-        <origin xyz="-0.957138 -0 0.2" rpy="0 0 0" />
-        <parent link="base_link" />
-        <child link="caster" />
-    </joint>
-    <!-- caster frontal wheel Link -->
-    <link name="caster">
-        <collision>
-            <geometry>
-                <sphere radius="0.2" />
-            </geometry>
-        </collision>
-        <visual>
-            <geometry>
-                <sphere radius="0.2" />
-            </geometry>
-            <material name="white" />
-        </visual>
-        <inertial>
-            <origin xyz="-0.957138 -0 0.2" rpy="0 0 0" />
-            <mass value="0.005" />
-            <inertia
-                ixx="0.1"
-                ixy="0.0"
-                ixz="0.0"
-                iyy="0.1"
-                iyz="0.0"
-                izz="0.1" />
-        </inertial>
-    </link>
     <gazebo>
         <!-- Joint state publisher -->

File: xacro/wheel.urdf.xacro (robot description, xacro)
@@ -31,5 +31,7 @@
                     <sphere radius="0.3" />
                 </geometry>
-                <material name="black" />
+                <material name="red">
+                    <color rgba="1 0 0 1" />
+                </material>
             </visual>
             <inertial>
@@ -43,4 +45,7 @@
             </inertial>
         </link>
+        <gazebo reference="${prefix}_wheel">
+            <material>Gazebo/Red</material>
+        </gazebo>
     </xacro:macro>
 </robot>
