Commit message: センサに色つけた

File: xacro/imu.xacro (robot description, xacro)
@@ -28,4 +28,7 @@
             </collision>
         </link>
+        <gazebo reference="imu_link">
+            <material>Gazebo/Blue</material>
+        </gazebo>
     </xacro:macro>
 </robot>

File: xacro/lidar.xacro (robot description, xacro)
@@ -23,4 +23,7 @@
             </visual>
         </link>
+        <gazebo reference="lidar_link">
+            <material>Gazebo/Red</material>
+        </gazebo>
     </xacro:macro>
 </robot>
