Commit message: caster修正

File: xacro/caster.urdf.xacro (robot description, xacro)
@@ -7,14 +7,24 @@
             <child link="caster" />
         </joint>
+        <transmission name="caster_trans" type="SimpleTransmission">
+            <type>transmission_interface/SimpleTransmission</type>
+            <actuator name="caster_motor">
+                <!-- ギア比 -->
+                <mechanicalReduction>1</mechanicalReduction>
+            </actuator>
+            <joint name="caster_joint">
+                <hardwareInterface>hardware_interface/VelocityJointInterface</hardwareInterface>
+            </joint>
+        </transmission>
         <!-- caster frontal wheel Link -->
         <link name="caster">
             <collision>
                 <geometry>
-                    <cylinder radius="0.05" length="0.03" />
+                    <sphere radius="0.05" />
                 </geometry>
             </collision>
             <visual>
                 <geometry>
-                    <cylinder radius="0.05" length="0.03" />
+                    <sphere radius="0.05" />
                 </geometry>
                 <material name="blue">
@@ -36,4 +46,7 @@
         <gazebo reference="caster">
             <material>Gazebo/Blue</material>
+            <!-- 摩擦係数はとりあえず0にして引っかからないようにする -->
+            <mu1>0.0</mu1>
+            <mu2>0.0</mu2>
         </gazebo>
     </xacro:macro>
