Commit message: サイズとか仮ぎめ

File: xacro/body.urdf.xacro (robot description, xacro)
@@ -5,13 +5,13 @@
         <link name="base_link">
             <collision>
-                <origin xyz="-0.151427 -0 0.5" rpy="0 0 0" />
+                <origin xyz="0 0 0.45" rpy="0 0 0" />
                 <geometry>
-                    <box size="2.01142 1 0.568726" />
+                    <box size="0.5 0.33 0.7" />
                 </geometry>
             </collision>
             <visual>
-                <origin xyz="-0.151427 -0 0.5" rpy="0 0 0" />
+                <origin xyz="0 0 0.45" rpy="0 0 0" />
                 <geometry>
-                    <box size="2.01142 1 0.568726" />
+                    <box size="0.5 0.33 0.7" />
                 </geometry>
                 <material name="white">
@@ -20,5 +20,5 @@
             </visual>
             <inertial>
-                <origin xyz="-0.151427 -0 0.5" rpy="0 0 0" />
+                <origin xyz="0 0 0.45" rpy="0 0 0" />
                 <mass value="1.14395" />
                 <inertia

File: xacro/caster.urdf.xacro (robot description, xacro)
@@ -1,7 +1,7 @@
 <?xml version="1.0"?>
 <robot xmlns:xacro="http://www.ros.org/wiki/xacro" name="caster">
-    <xacro:macro name="caster" params="parent">
+    <xacro:macro name="caster" params="parent xyz:='0 0 0' rpy:='0 0 0'">
         <joint name="caster_joint" type="fixed">
-            <origin xyz="-0.957138 -0 0.2" rpy="0 0 0" />
+            <origin xyz="${xyz}" rpy="${rpy}" />
             <parent link="${parent}" />
             <child link="caster" />
@@ -11,10 +11,10 @@
             <collision>
                 <geometry>
-                    <sphere radius="0.2" />
+                    <cylinder radius="0.05" length="0.03" />
                 </geometry>
             </collision>
             <visual>
                 <geometry>
-                    <sphere radius="0.2" />
+                    <cylinder radius="0.05" length="0.03" />
                 </geometry>
                 <material name="blue">

File: xacro/diff_drive_robot.urdf.xacro (robot description, xacro)
@@ -5,8 +5,12 @@
     <xacro:include filename="$(find ouagv_robot_description)/xacro/body.urdf.xacro" />
     <xacro:include filename="$(find ouagv_robot_description)/xacro/caster.urdf.xacro" />
+    <xacro:include filename="$(find ouagv_robot_description)/xacro/lidar.xacro" />
+    <xacro:include filename="$(find ouagv_robot_description)/xacro/imu.xacro" />
     <xacro:body />
-    <xacro:wheel prefix="left" parent="base_link" xyz="0.554283 0.625029 0.3" rpy="-1.5707 0 0" />
-    <xacro:wheel prefix="right" parent="base_link" xyz="0.554283 -0.625029 0.3" rpy="-1.5707 0 0" />
-    <xacro:caster parent="base_link" />
+    <xacro:wheel prefix="left" parent="base_link" xyz="0.125 0.21 0.125" rpy="-1.5707 0 0" />
+    <xacro:wheel prefix="right" parent="base_link" xyz="0.125 -0.21 0.125" rpy="-1.5707 0 0" />
+    <xacro:caster parent="base_link" xyz="-0.25 0 0.05" rpy="1.57 0 0" />
+    <xacro:lidar parent="base_link" xyz="0.3 0 0.2" rpy="0 0 0" />
+    <xacro:imu parent="base_link" xyz="0 0 0.8" rpy="0 0 0" />
     <xacro:diff_drive_control left_joint="left_wheel_joint" right_joint="right_wheel_joint" />
     <gazebo>

File: xacro/wheel.urdf.xacro (robot description, xacro)
@@ -24,10 +24,10 @@
             <collision>
                 <geometry>
-                    <sphere radius="0.3" />
+                    <cylinder radius="0.125" length="0.085" />
                 </geometry>
             </collision>
             <visual>
                 <geometry>
-                    <sphere radius="0.3" />
+                    <cylinder radius="0.125" length="0.085" />
                 </geometry>
                 <material name="red">

Commit message: fix mass

File: xacro/body.urdf.xacro (robot description, xacro)
@@ -21,12 +21,12 @@
             <inertial>
                 <origin xyz="0 0 0.45" rpy="0 0 0" />
-                <mass value="1.14395" />
+                <mass value="30" />
                 <inertia
-                    ixx="0.126164"
+                    ixx="0.1"
                     ixy="0.0"
                     ixz="0.0"
-                    iyy="0.416519"
+                    iyy="0.1"
                     iyz="0.0"
-                    izz="0.481014" />
+                    izz="0.1" />
             </inertial>
         </link>

File: xacro/caster.urdf.xacro (robot description, xacro)
@@ -24,5 +24,5 @@
             <inertial>
                 <origin xyz="-0.957138 -0 0.2" rpy="0 0 0" />
-                <mass value="0.005" />
+                <mass value="1.1" />
                 <inertia
                     ixx="0.1"

File: xacro/imu.xacro (robot description, xacro)
@@ -12,5 +12,5 @@
             <visual>
                 <inertial>
-                    <mass value="0.3" />
+                    <mass value="0.03" />
                     <inertia ixx="0.01" ixy="0.0" ixz="0" iyy="0.01" iyz="0" izz="0.01" />
                 </inertial>

File: xacro/lidar.xacro (robot description, xacro)
@@ -11,5 +11,5 @@
         <link name="lidar_link">
             <inertial>
-                <mass value="0.5" />
+                <mass value="0.3" />
                 <inertia ixx="0.01" ixy="0.0" ixz="0" iyy="0.01" iyz="0" izz="0.01" />
             </inertial>

File: xacro/wheel.urdf.xacro (robot description, xacro)
@@ -36,11 +36,11 @@
             </visual>
             <inertial>
-                <mass value="2" />
-                <inertia ixx="0.145833"
+                <mass value="1.7" />
+                <inertia ixx="0.1"
                     ixy="0.0"
                     ixz="0.0"
-                    iyy="0.145833"
+                    iyy="0.1"
                     iyz="0.0"
-                    izz="0.125" />
+                    izz="0.1" />
             </inertial>
         </link>

Commit message: 追加

File: xacro/body.urdf.xacro (robot description, xacro)
@@ -23,10 +23,10 @@
                 <mass value="30" />
                 <inertia
-                    ixx="0.1"
+                    ixx="0.6"
                     ixy="0.0"
                     ixz="0.0"
-                    iyy="0.1"
+                    iyy="0.6"
                     iyz="0.0"
-                    izz="0.1" />
+                    izz="0.6" />
             </inertial>
         </link>

File: xacro/lidar.xacro (robot description, xacro)
@@ -48,5 +48,5 @@
                     <range>
                         <min>0.1</min>
-                        <max>30.0</max>
+                        <max>15.0</max>
                         <resolution>0.01</resolution>
                     </range>

File: xacro/wheel.urdf.xacro (robot description, xacro)
@@ -36,11 +36,11 @@
             </visual>
             <inertial>
-                <mass value="1.7" />
-                <inertia ixx="0.1"
+                <mass value="3.0" />
+                <inertia ixx="0.3"
                     ixy="0.0"
                     ixz="0.0"
-                    iyy="0.1"
+                    iyy="0.3"
                     iyz="0.0"
-                    izz="0.1" />
+                    izz="0.3" />
             </inertial>
         </link>
